File: Eagle Files/Fab House Design/AP_AT42QT2120.sch (EAGLE design)
At the start: 12 parts

Commit message: board tags
Parts:
- removed R24, R25: 4.7k, rcl:R-US_R1206
- added R1, R2: 4.7k, rcl:R-US_R1206
- U1: value AT42QT2120-SU -> AT42QT2120
- renumbered C2 to C1, JP1 to TOUCH, R21 to R4, R22 to R5, R23 to R6, R9 to R3, U$1 to U1
Connections:
- net +3V3: now also R1.1, R2.1; no longer R7.1, R8.1
- net N$10: now also R8.1; no longer R25.1
- net N$11: now also R7.1; no longer R24.1
- net N$25: now also R2.2; no longer R7.2
- net N$27: now also R1.2; no longer R8.2
- net N$8: now also R7.2; no longer R24.2
- net N$9: now also R8.2; no longer R25.2
Other:
- moved on the sheet: R7, R8
