File: Eagle Files/Fab House Design/AP_AT42QT2120.brd (EAGLE design)
At the start: 20 x 40 mm, 12 parts

Commit message: board tags
Parts:
- removed JP1: PINHD-1X5, Connector:1X05
- removed R24, R25: 4.7k, rcl:R1206
- removed R9: 47k, rcl:R1206
- added R1, R2: 4.7k, rcl:R1206
- added R3: 47k, rcl:R1206
- added TOUCH: PINHD-1X5, Connector:1X05
- U1: value AT42QT2120-SU -> AT42QT2120
- moved R8 22.9 mm to (17.0, 8.47), turned to 90 degrees
- moved R7 18.2 mm to (14.4, 8.47), turned to 90 degrees
- moved IO 2.88 mm to (10.0, 37.3)
- renumbered C2 to C1, R21 to R4, R22 to R5, R23 to R6, U$1 to U1
Connections:
- removed net N$13: JP1.4, R5.1
- new net N$2: R5.1, TOUCH.4
- net +3V3: now also R1.1, R2.1, R3.1; no longer R7.1, R8.1, R9.1
- net N$10: now also R8.1, TOUCH.1; no longer JP1.1, R25.1
- net N$11: now also R7.1, TOUCH.2; no longer JP1.2, R24.1
- net N$12: now also TOUCH.3; no longer JP1.3
- net N$14: now also TOUCH.5; no longer JP1.5
- net N$25: now also R2.2; no longer R7.2
- net N$26: now also R3.2; no longer R9.2
- net N$27: now also R1.2; no longer R8.2
- net N$8: now also R7.2; no longer R24.2
- net N$9: now also R8.2; no longer R25.2
Routing:
- net N$13: track 2.96 -> 0.00 mm
- net N$25: track 19.0 -> 21.3 mm
- net N$26: track 27.3 -> 25.1 mm
- net +3V3: track 21.7 -> 23.5 mm
- net N$27: track 15.7 -> 17.4 mm
- net N$1: track 16.0 -> 17.7 mm
- net N$12: track 2.91 -> 4.60 mm
- net N$11: track 2.87 -> 4.55 mm
- net N$10: track 2.88 -> 4.53 mm
- net N$14: track 2.90 -> 4.55 mm

Commit message: finals
Parts:
- moved IO 5.20 mm to (10.0, 42.5)
- moved C1 4.41 mm to (16.7, 22.9)
- moved R1 3.00 mm to (16.5, 34.4)
- moved R2 3.00 mm to (16.6, 31.9)
- moved R3 3.00 mm to (16.6, 29.5)
- moved U1 2.72 mm to (3.00, 16.4)
- moved R7 1.73 mm to (14.1, 10.2)
- moved R8 1.73 mm to (16.7, 10.2)
- moved R6 1.63 mm to (11.6, 10.1)
- moved R5 1.55 mm to (8.99, 10.0)
- moved R4 1.53 mm to (6.49, 10.0)
- moved TOUCH 1.08 mm to (11.6, 3.59)
Routing:
- net N$2: track 0.00 -> 5.00 mm
- net N$1: track 17.7 -> 20.5 mm
- net N$26: track 25.1 -> 27.6 mm
- net N$27: track 17.4 -> 19.9 mm
- net N$25: track 21.3 -> 23.4 mm
- net N$5: track 4.76 -> 6.56 mm
- net N$6: track 4.13 -> 5.40 mm
- net N$10: track 4.53 -> 5.17 mm
- net N$11: track 4.55 -> 5.17 mm
- net N$12: track 4.60 -> 5.11 mm
- added copper zone on layer 1, net GND
Other:
- board size 20 x 40 mm -> 20 x 46 mm
- board text added: "3V3"
- board text added: "Cap Touch Rev A"
- board text added: "GND"
- board text added: "INT"
- board text added: "K3"
- board text added: "K4"
- board text added: "RST"
- board text added: "S0"
- board text added: "S1"
- board text added: "S2"
- board text added: "SCL"
- board text added: "SDA"
