File: Eagle Files/Fab House Design/touch_w_scroll.brd (EAGLE design)
At the start: 18 x 85 mm, 4 parts

Commit message: finals
Parts:
- moved JP1 1.46 mm to (8.40, 81.4)
Routing:
- net N$1: track 12.7 -> 13.9 mm
- net N$2: track 98.3 -> 99.5 mm
- net N$4: track 62.6 -> 63.6 mm
- net N$5: track 46.6 -> 47.6 mm
- net N$3: track 85.0 -> 86.0 mm
Other:
- board text added: "Cap Touch Rev A"
